File: projects/FDevT/02 hardware/03 sheet/FDevT.sch (EAGLE design)
At the start: 19 parts, among them IC2 LP2950

Commit message: final Version
Parts:
- added SG1: F/TMB, buzzer:F/TMB
- added STEPPER: TBB6612, TBB6612d:TBB6612
- added U$4: STEPUP, AMESYS_neu:STEPUP
- added X4: OUTB, con-phoenix-254:MPT2
- C1, C4, C6, C7, C9: value (none) -> 100n
- C2, C3, C5, C8: value (none) -> 10µ
- X1: value (none) -> IN
- X2: value (none) -> Motor
- X3: value (none) -> OUTA
Connections:
- removed net R_CHANGE: BOARD1.D2
- new net AIN1: BOARD1.D2, STEPPER.AIN2
- new net AIN2: BOARD1.D4, STEPPER.AIN1
- new net N$3: STEPPER.A1, X3-2.1
- new net N$4: STEPPER.A2, X3-1.1
- new net N$5: BOARD1.D5, STEPPER.BIN1
- new net N$6: BOARD1.D18, STEPPER.BIN2
- new net N$7: BOARD1.D19, STEPPER.PWMB
- new net N$8: STEPPER.B2, X4-2.1
- new net N$9: STEPPER.B1, X4-1.1
- net +12V: now also STEPPER.VM, U$4.IN
- net +3V3: now also STEPPER.STBY, STEPPER.VCC1
- net +5V: now also U$4.OUT
- net BEEP: now also BOARD1.D17, SG1.+; no longer BOARD1.D4
- net GND: now also SG1.-, STEPPER.GND1, STEPPER.GND3, U$4.GND
- net PWM: now also STEPPER.PWMA
Other:
- note added: "AIN1 high, AIN2 low --> CW"
- note added: "AIN1 low, AIN2 high --> CCW"
- moved on the sheet: C8, C9, X1-1, X1-2, X2-1, X2-2, X2-3, X3-1, X3-2
